Commit message: docs: RRC Lite IMU 회전 방향 확인 (반시계 = +, ROS 규칙 일치)
- 보드 단독 시험: 반시계 90° -> +82.7°, 시계 90° -> -93.6°
- URDF imu_yaw 주석에 확인 결과 기록 (장착 후 방향 재확인 필요)

Co-Authored-By: Claude Opus 5.5 <noreply@anthropic.com>

File: ros2_ws/src/poli_description/urdf/poli.urdf.xacro (robot description, xacro)
@@ -33,5 +33,5 @@
   <xacro:property name="imu_y" value="0.0"/>                 <!-- TODO_MEASURE -->
   <xacro:property name="imu_h" value="0.05"/>                <!-- SIM_ONLY -->
-  <xacro:property name="imu_yaw" value="0.0"/>               <!-- 보드 방향. 좌회전 시 gz > 0 이 되게 (TODO_MEASURE) -->
+  <xacro:property name="imu_yaw" value="0.0"/>               <!-- 보드 방향. 2026-10-06 보드 단독: 반시계 = +gz 확인. 장착 방향에 따라 재확인 (TODO_MEASURE) -->
   <!-- ===== 카메라 (Raspberry Pi AI Camera, CAM0) ===== -->
   <xacro:property name="camera_x" value="0.09"/>             <!-- SIM_ONLY -->

Commit message: 집게 서보를 RRC Lite PWM 포트로 이전, 제품 사양서_E 대조 반영
- 사양서_E 연결 계획(PWM 서보 제어 = 그리퍼)과 팀 결정에 따라 DS3218을 Mega D9에서
  RRC Lite PWM 서보 포트로 옮김. rrc_adapter_node/fake_rrc_node가 /gripper/command,
  /gripper/state를 맡는다 (토픽 약속은 그대로). mega_bridge_node는 초음파만.
- rrc_protocol: func 4 PWM 서보 설정/읽기 frame, gripper.py: 상태 판단(open/closed/moving).
- 첫 명령 전에는 서보 명령을 보내지 않음(규정 3.5.6). RRC가 전원 켤 때 1500 us를 내므로
  열림 = 1500 us. 서보 포트 전원 점퍼 5V 필수(문서·설정 주석).
- max_wheel_rpm 330 -> 250 (사양서 정격 동작점), URDF wheel_width 0.026 (바퀴 65x26 mm).
- AGENTS.md 1장: 제품 사양서를 부품 기준으로 대조하는 규칙. hardware_reference 0장:
  일치 항목, 변경 내역, 사양서 작성자 확인 요청 목록. Pi 전원 방법은 미정으로 기록.

Co-Authored-By: Claude Opus 5.5 <noreply@anthropic.com>

File: ros2_ws/src/poli_description/urdf/poli.urdf.xacro (robot description, xacro)
@@ -13,6 +13,6 @@
 <robot name="poli" xmlns:xacro="http://www.ros.org/wiki/xacro">
   <!-- ===== 차체 ===== -->
-  <xacro:property name="wheel_radius" value="0.0325"/>       <!-- 65 mm 바퀴. 주행 시험으로 보정 (TODO_MEASURE) -->
-  <xacro:property name="wheel_width" value="0.027"/>         <!-- SIM_ONLY -->
+  <xacro:property name="wheel_radius" value="0.0325"/>       <!-- 바퀴 Ø65 mm (제품 사양서_E). 주행 시험으로 보정 (TODO_MEASURE) -->
+  <xacro:property name="wheel_width" value="0.026"/>         <!-- 고무 바퀴 Ø65 × 26 mm (제품 사양서_E) -->
   <xacro:property name="wheel_separation" value="0.18"/>     <!-- 좌우 바퀴 중심 간 거리 (TODO_MEASURE, hardware.yaml과 같게) -->
   <xacro:property name="body_length" value="0.20"/>          <!-- 집게 제외 차체 길이 (TODO_MEASURE) -->

Commit message: poli_hardware: RRC 노드 삭제, mega_bridge_node가 주행·센서·집게 담당
Mega 포트 하나를 한 노드만 열 수 있어 주행(MDD10)·엔코더·IMU·초음파·집게를
mega_bridge_node 하나로 합쳤다. 토픽 이름·형식·frame_id는 그대로.

- drive_node.py: 공통 노드 (cmd_vel 0.3 s timeout, 25 Hz 연속 명령 유지)
- mega_bridge_node: $DRV 전송, $ENC로 /odom_raw (엔코더 기반), $IMU로 /imu/data
- fake_mega_node: 부품 없이 같은 토픽
- rrc_node.py, rrc_protocol.py, gripper.py와 테스트 삭제, /battery_state 없앰
- mega_protocol: ENC/IMU/DRV/PWM, WheelSpeedEstimator + 테스트
- min_wheel_speed 0.25 유지 (turn_pulse.HW_MIN_WHEEL_SPEED와 맞춰야 함)
- scripts: pi_comm_check·wheel_test를 Mega 기준으로, pc_serial_tester에 방향 시험(f/b)
- URDF imu_link 주석을 BNO085로

Co-Authored-By: Claude Opus 5.5 <noreply@anthropic.com>

File: ros2_ws/src/poli_description/urdf/poli.urdf.xacro (robot description, xacro)
@@ -29,9 +29,9 @@
   <xacro:property name="lidar_mount_h" value="${body_top_h}"/>  <!-- 장착면 지면 높이 (TODO_MEASURE) -->
   <xacro:property name="lidar_yaw" value="0.0"/>             <!-- 스캔 0도 방향이 정면이 되게 (TODO_MEASURE) -->
-  <!-- ===== IMU (RRC Lite 내장 QMI8658) ===== -->
-  <xacro:property name="imu_x" value="0.0"/>                 <!-- RRC Lite 보드 위치 (TODO_MEASURE) -->
+  <!-- ===== IMU (BNO085, Mega I2C. 2026-10-29 RRC Lite 내장 IMU에서 변경) ===== -->
+  <xacro:property name="imu_x" value="0.0"/>                 <!-- BNO085 보드 위치 (TODO_MEASURE) -->
   <xacro:property name="imu_y" value="0.0"/>                 <!-- TODO_MEASURE -->
   <xacro:property name="imu_h" value="0.05"/>                <!-- SIM_ONLY -->
-  <xacro:property name="imu_yaw" value="0.0"/>               <!-- 보드 방향. 2026-10-06 보드 단독: 반시계 = +gz 확인. 장착 방향에 따라 재확인 (TODO_MEASURE) -->
+  <xacro:property name="imu_yaw" value="0.0"/>               <!-- 보드 방향. 로봇을 반시계로 돌릴 때 /imu/data gz가 +가 되게 (TODO_MEASURE) -->
   <!-- ===== 카메라 (Raspberry Pi AI Camera, CAM0) ===== -->
   <xacro:property name="camera_x" value="0.09"/>             <!-- SIM_ONLY -->

Commit message: 로봇 실측 치수 반영 (URDF, wheel_separation, 크기 규정 점검)
2026-10-30 줄자 실측: 길이 330(집게 제외 210), 폭 305(바퀴 제외 220) mm,
바퀴 축 = 뒤끝에서 160 mm, 볼캐스터 = 뒤끝 30 mm, LiDAR·카메라 좌우 위치.
- wheel_separation 0.18(임시값) -> 0.279 (305 - 바퀴 폭 26). 회전 보정 필요
- URDF 차체·캐스터·LiDAR·카메라·집게 위치를 실측값으로 (LiDAR 앞뒤는 사진 추정, TODO_MEASURE)
- rules_compliance 2.2.1: 감싸는 원 약 390 mm 추정, 집게 연 상태 실측 필요

Co-Authored-By: Claude Opus 5.5 <noreply@anthropic.com>

File: ros2_ws/src/poli_description/urdf/poli.urdf.xacro (robot description, xacro)
@@ -15,16 +15,18 @@
   <xacro:property name="wheel_radius" value="0.0325"/>       <!-- 바퀴 Ø65 mm (제품 사양서_E). 주행 시험으로 보정 (TODO_MEASURE) -->
   <xacro:property name="wheel_width" value="0.026"/>         <!-- 고무 바퀴 Ø65 × 26 mm (제품 사양서_E) -->
-  <xacro:property name="wheel_separation" value="0.18"/>     <!-- 좌우 바퀴 중심 간 거리 (TODO_MEASURE, hardware.yaml과 같게) -->
-  <xacro:property name="body_length" value="0.20"/>          <!-- 집게 제외 차체 길이 (TODO_MEASURE) -->
-  <xacro:property name="body_width" value="0.22"/>           <!-- 외곽 폭 220 mm (집게 연 상태 제공값) -->
+  <xacro:property name="wheel_separation" value="0.279"/>    <!-- 바퀴 포함 폭 305 - 바퀴 폭 26 (2026-10-30 줄자). 회전 시험으로 보정 (TODO_MEASURE, hardware.yaml과 같게) -->
+  <xacro:property name="body_length" value="0.21"/>          <!-- 집게 제외 차체 길이 210 mm (2026-10-30 실측) -->
+  <xacro:property name="body_width" value="0.22"/>           <!-- 바퀴 제외 차체 폭 220 mm (2026-10-30 실측) -->
   <xacro:property name="body_bottom_h" value="0.02"/>        <!-- 차체 바닥의 지면 높이 (TODO_MEASURE) -->
   <xacro:property name="body_top_h" value="0.14"/>           <!-- 차체 윗면의 지면 높이 (TODO_MEASURE) -->
-  <xacro:property name="body_center_x" value="0.0"/>         <!-- 바퀴 축 기준 차체 중심 앞뒤 위치 (TODO_MEASURE) -->
-  <xacro:property name="caster_x" value="-0.08"/>            <!-- 뒤 지지점(캐스터) 위치 (TODO_MEASURE) -->
+  <!-- 2026-10-30 실측: 바퀴 축 = 차체 뒤끝에서 160 mm, 볼캐스터 = 뒤끝에서 30 mm (좌우 가운데) -->
+  <xacro:property name="axle_from_rear" value="0.16"/>
+  <xacro:property name="body_center_x" value="${body_length / 2 - axle_from_rear}"/>  <!-- = -0.055 -->
+  <xacro:property name="caster_x" value="${0.03 - axle_from_rear}"/>                   <!-- = -0.13 -->
   <!-- ===== LiDAR (RPLIDAR C1) =====
        laser 높이 = 장착면 높이 + 0.0298. 외벽·장애물(0.20 m)보다 낮아야 한다.
        frame 이름 'laser'는 sllidar_ros2 기본값·poli_navigation fake_scan과 같다. -->
-  <xacro:property name="lidar_x" value="0.0"/>               <!-- TODO_MEASURE (scan_to_grid.py LASER_OFFSET과 맞출 것) -->
-  <xacro:property name="lidar_y" value="0.0"/>               <!-- TODO_MEASURE -->
+  <xacro:property name="lidar_x" value="${0.08 - axle_from_rear}"/>  <!-- 중심이 뒤끝에서 약 80 mm: 사진 추정 (TODO_MEASURE, scan_to_grid.py LASER_OFFSET과 맞출 것) -->
+  <xacro:property name="lidar_y" value="${body_width / 2 - 0.115}"/>  <!-- 중심이 좌측 끝에서 115 mm (2026-10-30 실측) = 오른쪽 5 mm -->
   <xacro:property name="lidar_mount_h" value="${body_top_h}"/>  <!-- 장착면 지면 높이 (TODO_MEASURE) -->
   <xacro:property name="lidar_yaw" value="0.0"/>             <!-- 스캔 0도 방향이 정면이 되게 (TODO_MEASURE) -->
@@ -35,5 +37,6 @@
   <xacro:property name="imu_yaw" value="0.0"/>               <!-- 보드 방향. 로봇을 반시계로 돌릴 때 /imu/data gz가 +가 되게 (TODO_MEASURE) -->
   <!-- ===== 카메라 (Raspberry Pi AI Camera, CAM0) ===== -->
-  <xacro:property name="camera_x" value="0.09"/>             <!-- SIM_ONLY -->
+  <xacro:property name="camera_x" value="${body_center_x + body_length / 2}"/>  <!-- 2층 판 앞끝 (사진 확인) -->
+  <xacro:property name="camera_y" value="${body_width / 2 - 0.12}"/>  <!-- 좌측 끝에서 120 mm (2026-10-30 실측) = 오른쪽 10 mm -->
   <xacro:property name="camera_h" value="0.12"/>             <!-- SIM_ONLY -->
   <xacro:property name="camera_pitch" value="0.26"/>         <!-- 아래로 숙인 각 (약 15도, SIM_ONLY) -->
@@ -48,5 +51,6 @@
   <xacro:property name="us_side_y" value="${body_width / 2}"/>
   <!-- ===== 집게 (Byte Robot Claw 125mm, 들어 올리기 없음) ===== -->
-  <xacro:property name="gripper_x" value="${body_center_x + body_length / 2 + 0.03}"/>  <!-- SIM_ONLY -->
+  <xacro:property name="gripper_len" value="0.12"/>          <!-- 차체 앞으로 튀어나온 길이: 전체 330 - 차체 210 (2026-10-30 실측, 닫힘) -->
+  <xacro:property name="gripper_x" value="${body_center_x + body_length / 2 + gripper_len / 2}"/>
   <xacro:property name="gripper_h" value="0.05"/>            <!-- SIM_ONLY -->
   <material name="dark"><color rgba="0.2 0.2 0.2 1.0"/></material>
@@ -124,5 +128,5 @@
     <parent link="base_link"/>
     <child link="camera_link"/>
-    <origin xyz="${camera_x} 0 ${camera_h - wheel_radius}" rpy="0 ${camera_pitch} 0"/>
+    <origin xyz="${camera_x} ${camera_y} ${camera_h - wheel_radius}" rpy="0 ${camera_pitch} 0"/>
   </joint>
   <xacro:macro name="ultrasonic" params="name x y h yaw">
@@ -145,5 +149,5 @@
   <link name="gripper_link">
     <visual>
-      <geometry><box size="0.06 0.125 0.04"/></geometry>
+      <geometry><box size="${gripper_len} 0.125 0.04"/></geometry>
       <material name="dark"/>
     </visual>

Commit message: MPU6050 imu_node 추가: /imu/data를 파이 I2C IMU가 발행 (RRC 내장 IMU 대체)
RRC Lite 소손(2026-10-29)으로 IMU를 파이 GPIO 소프트웨어 I2C 버스 3(15·16번 핀)에 직접 연결.
3번 핀이 사용 중이라 하드웨어 I2C 대신 i2c-gpio 오버레이를 쓴다. 시작 때 자이로 영점 후 발행,
토픽 계약(/imu/data, imu_link, 50 Hz)은 그대로. rrc_adapter_node는 publish_imu: false.
실기 미검증(가짜 센서로만 확인).

Co-Authored-By: Claude Opus 5.5 <noreply@anthropic.com>

File: ros2_ws/src/poli_description/urdf/poli.urdf.xacro (robot description, xacro)
@@ -30,8 +30,9 @@
   <xacro:property name="lidar_yaw" value="0.0"/>             <!-- 스캔 0도 방향이 정면이 되게 (TODO_MEASURE) -->
   <!-- ===== IMU (RRC Lite 내장 QMI8658) ===== -->
-  <xacro:property name="imu_x" value="0.0"/>                 <!-- RRC Lite 보드 위치 (TODO_MEASURE) -->
-  <xacro:property name="imu_y" value="0.0"/>                 <!-- TODO_MEASURE -->
-  <xacro:property name="imu_h" value="0.05"/>                <!-- SIM_ONLY -->
-  <xacro:property name="imu_yaw" value="0.0"/>               <!-- 보드 방향. 2026-10-06 보드 단독: 반시계 = +gz 확인. 장착 방향에 따라 재확인 (TODO_MEASURE) -->
+  <!-- 2026-10-30 RRC Lite 내장 IMU -> MPU6050(GY-521, 파이 I2C). 모듈의 X 화살표가 로봇 앞, 칩이 위면 yaw 0 -->
+  <xacro:property name="imu_x" value="0.0"/>                 <!-- MPU6050 위치, base_link 기준 앞(+) (TODO_MEASURE) -->
+  <xacro:property name="imu_y" value="0.0"/>                 <!-- 왼쪽(+) (TODO_MEASURE) -->
+  <xacro:property name="imu_h" value="0.05"/>                <!-- 바닥에서 높이 (SIM_ONLY) -->
+  <xacro:property name="imu_yaw" value="0.0"/>               <!-- X 화살표가 앞에서 반시계로 돈 각 [rad]. 제자리 반시계 회전 = +gz 확인 (TODO_MEASURE) -->
   <!-- ===== 카메라 (Raspberry Pi AI Camera, CAM0) ===== -->
   <xacro:property name="camera_x" value="0.09"/>             <!-- SIM_ONLY -->

Commit message: IMU를 BNO085 -> MPU-6050으로 변경 (펌웨어, Pi 파서, 문서)
팀이 실제로 단 IMU는 MPU-6050 (2026-10-30 확인).
- 펌웨어 imu.cpp: Wire로 MPU-6050 직접 읽기 (라이브러리 없음). 주소 0x68,
  자이로 ±500 dps, 가속도 ±4 g, 저역 필터 44 Hz, 켤 때 1초 자이로 영점.
  읽기가 0.2 s 넘게 실패하면 $IMU를 멈춤. SIM_IMU 기본 0
- $IMU 형식은 그대로, MPU-6050은 방향이 없으므로 q = 0,0,0,0
- Pi: ImuPacket.to_si()가 q = 0이면 None -> /imu/data orientation 없음 (covariance -1)
- 문서·AGENTS.md의 BNO085 표기를 MPU-6050으로, SparkFun BNO080 라이브러리 설치 줄 삭제

Co-Authored-By: Claude Opus 5.5 <noreply@anthropic.com>

File: ros2_ws/src/poli_description/urdf/poli.urdf.xacro (robot description, xacro)
@@ -31,6 +31,6 @@
   <xacro:property name="lidar_mount_h" value="${body_top_h}"/>  <!-- 장착면 지면 높이 (TODO_MEASURE) -->
   <xacro:property name="lidar_yaw" value="0.0"/>             <!-- 스캔 0도 방향이 정면이 되게 (TODO_MEASURE) -->
-  <!-- ===== IMU (BNO085, Mega I2C. 2026-10-29 RRC Lite 내장 IMU에서 변경) ===== -->
-  <xacro:property name="imu_x" value="0.0"/>                 <!-- BNO085 보드 위치 (TODO_MEASURE) -->
+  <!-- ===== IMU (MPU-6050, Mega I2C. 2026-10-30) ===== -->
+  <xacro:property name="imu_x" value="0.0"/>                 <!-- MPU-6050 칩 위치 (TODO_MEASURE) -->
   <xacro:property name="imu_y" value="0.0"/>                 <!-- TODO_MEASURE -->
   <xacro:property name="imu_h" value="0.05"/>                <!-- SIM_ONLY -->
